File: hardware/vco/vco.kicad_pcb (KiCad board)
At the start: 2 copper layers, 71.9 x 100 mm, 109 parts, among them J1 AudioJack2, J2 AudioJack2, J3 AudioJack2, J4 AudioJack2, J5 AudioJack2, J6 AudioJack2, J7 AudioJack2, J8 16 Pin IDC, Q1 BC557B, Q2 BC547B, U1 TL074, U2 TL074, U3 TL074

Commit message: Polish for submission
Parts:
- added C13: 10u, Capacitor_THT:CP_Radial_D4.0mm_P2.00mm, B.Cu at (136.2, 90.2)
- added C14: 22u, Capacitor_THT:CP_Radial_D4.0mm_P2.00mm, B.Cu at (136.2, 94.8)
- added C15: 10u, Capacitor_THT:CP_Radial_D4.0mm_P2.00mm, B.Cu at (161.6, 91.7)
- added REF**: MountingHole_3.2mm_M3, MountingHole:MountingHole_3.2mm_M3, F.Cu at (186.9, 20.0)
- added U4: AMS1117-2.5, Package_TO_SOT_SMD:SOT-223-3_TabPin2, B.Cu at (141.9, 92.8)
- added U5: TC7660, TC7660:DIL08, B.Cu at (152.8, 91.4)
- D10, D11, D12, D13, D14, D15, D4, D5, D6, D7, D8, D9, R33, R34, R35, R36, R37, R38, R39, R40, R41, R42, R43, R44, R45, R46, R47, R48, R49, R50, R51, R52, R53: moved to B.Cu
- moved R53 98.6 mm to (165.8, 97.9)
- moved R39 96.0 mm to (171.6, 82.6), turned to 180 degrees
- moved R45 95.8 mm to (171.6, 90.7), turned to 180 degrees
- moved R48 95.7 mm to (171.6, 94.7), turned to 180 degrees
- moved R42 92.9 mm to (171.6, 86.6), turned to 180 degrees
- moved R33 89.9 mm to (169.6, 75.9)
- moved R34 88.3 mm to (171.7, 79.0), turned to 180 degrees
- moved R49 82.4 mm to (184.5, 102.0), turned to -90 degrees
- moved R46 82.2 mm to (186.7, 94.7), turned to 180 degrees
- moved R50 82.2 mm to (186.7, 97.7), turned to 180 degrees
- moved D15 81.8 mm to (174.3, 101.8)
- moved R38 81.2 mm to (189.9, 78.2), turned to -90 degrees
- moved D13 80.6 mm to (174.3, 96.7)
- moved R36 80.3 mm to (186.7, 76.0), turned to 180 degrees
- moved D11 79.6 mm to (174.3, 91.6)
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Routing:
- net +12V: track 0.00 -> 189.6 mm, vias 0 -> 2
- net -12V: track 0.00 -> 163.1 mm, vias 0 -> 5
- net /SAW: track 0.00 -> 135.6 mm
- net Net-(Q1-B): track 0.00 -> 117.9 mm, vias 0 -> 2
- net /PWM: track 0.00 -> 71.6 mm
- net Net-(D1-K): track 0.00 -> 69.7 mm, vias 0 -> 2
- net +2V5: track 0.00 -> 64.9 mm, vias 0 -> 2
- net Net-(D2-A): track 0.00 -> 64.4 mm
- net Net-(D14-A): track 0.00 -> 52.6 mm
- net /TRI: track 0.00 -> 49.9 mm, vias 0 -> 1
- net Net-(U2A-+): track 0.00 -> 46.7 mm, vias 0 -> 1
- net Net-(R51-Pad2): track 0.00 -> 46.2 mm
- net -2V5: track 0.00 -> 41.8 mm, vias 0 -> 2
- net GND: track 0.00 -> 34.5 mm, vias 0 -> 148
- net /PWM_CV: track 0.00 -> 22.6 mm
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- added copper zone on B.Cu, net GND
- removed copper zone on B.Cu, net (none)
Other:
- board text added: "1V/O"
- board text added: "FM"
- board text added: "FM SCALE"
- board text added: "PITCH"
- board text added: "PWM"
- board text added: "PWM SCALE"
- board text added: "SAW"
- board text added: "SIN"
- board text added: "TRI"
- board text added: "TRI OFF"
